Commit message: ur3

File: urdfs/ur3/ur3.urdf.xacro (robot description, xacro)
@@ -4,6 +4,6 @@
   Author: Felix Messmer
 -->
-  <xacro:include filename="$(find ur_description)/urdf/ur.transmission.xacro" />
-  <xacro:include filename="$(find ur_description)/urdf/ur.gazebo.xacro" />
+  <xacro:include filename="ur.transmission.xacro" />
+  <xacro:include filename="ur.gazebo.xacro" />
    <xacro:macro name="cylinder_inertial" params="radius length mass *origin">
     <inertial>
@@ -64,13 +64,13 @@
       <visual>
         <geometry>
-          <mesh filename="package://ur_description/meshes/ur3/visual/base.dae"/>
-        </geometry>
-        <material name="LightGrey">
-          <color rgba="0.7 0.7 0.7 1.0"/>
-        </material>
-      </visual>
-      <collision>
-        <geometry>
-          <mesh filename="package://ur_description/meshes/ur3/collision/base.stl"/>
+          <mesh filename="visual/base.dae"/>
+        </geometry>
+        <material name="LightGrey">
+          <color rgba="0.7 0.7 0.7 1.0"/>
+        </material>
+      </visual>
+      <collision>
+        <geometry>
+          <mesh filename="collision/base.stl"/>
         </geometry>
       </collision>
@@ -101,13 +101,13 @@
       <visual>
         <geometry>
-          <mesh filename="package://ur_description/meshes/ur3/visual/shoulder.dae"/>
-        </geometry>
-        <material name="LightGrey">
-          <color rgba="0.7 0.7 0.7 1.0"/>
-        </material>
-      </visual>
-      <collision>
-        <geometry>
-          <mesh filename="package://ur_description/meshes/ur3/collision/shoulder.stl"/>
+          <mesh filename="visual/shoulder.dae"/>
+        </geometry>
+        <material name="LightGrey">
+          <color rgba="0.7 0.7 0.7 1.0"/>
+        </material>
+      </visual>
+      <collision>
+        <geometry>
+          <mesh filename="collision/shoulder.stl"/>
         </geometry>
       </collision>
@@ -138,13 +138,13 @@
       <visual>
         <geometry>
-          <mesh filename="package://ur_description/meshes/ur3/visual/upperarm.dae"/>
-        </geometry>
-        <material name="LightGrey">
-          <color rgba="0.7 0.7 0.7 1.0"/>
-        </material>
-      </visual>
-      <collision>
-        <geometry>
-          <mesh filename="package://ur_description/meshes/ur3/collision/upperarm.stl"/>
+          <mesh filename="visual/upperarm.dae"/>
+        </geometry>
+        <material name="LightGrey">
+          <color rgba="0.7 0.7 0.7 1.0"/>
+        </material>
+      </visual>
+      <collision>
+        <geometry>
+          <mesh filename="collision/upperarm.stl"/>
         </geometry>
       </collision>
@@ -175,13 +175,13 @@
       <visual>
          <geometry>
-          <mesh filename="package://ur_description/meshes/ur3/visual/forearm.dae"/>
-        </geometry>
-        <material name="LightGrey">
-          <color rgba="0.7 0.7 0.7 1.0"/>
-        </material>
-      </visual>
-      <collision>
-        <geometry>
-          <mesh filename="package://ur_description/meshes/ur3/collision/forearm.stl"/>
+          <mesh filename="visual/forearm.dae"/>
+        </geometry>
+        <material name="LightGrey">
+          <color rgba="0.7 0.7 0.7 1.0"/>
+        </material>
+      </visual>
+      <collision>
+        <geometry>
+          <mesh filename="collision/forearm.stl"/>
         </geometry>
       </collision>
@@ -212,13 +212,13 @@
       <visual>
         <geometry>
-          <mesh filename="package://ur_description/meshes/ur3/visual/wrist1.dae"/>
-        </geometry>
-        <material name="LightGrey">
-          <color rgba="0.7 0.7 0.7 1.0"/>
-        </material>
-      </visual>
-      <collision>
-        <geometry>
-          <mesh filename="package://ur_description/meshes/ur3/collision/wrist1.stl"/>
+          <mesh filename="visual/wrist1.dae"/>
+        </geometry>
+        <material name="LightGrey">
+          <color rgba="0.7 0.7 0.7 1.0"/>
+        </material>
+      </visual>
+      <collision>
+        <geometry>
+          <mesh filename="collision/wrist1.stl"/>
         </geometry>
       </collision>
@@ -249,13 +249,13 @@
       <visual>
         <geometry>
-          <mesh filename="package://ur_description/meshes/ur3/visual/wrist2.dae"/>
-        </geometry>
-        <material name="LightGrey">
-          <color rgba="0.7 0.7 0.7 1.0"/>
-        </material>
-      </visual>
-      <collision>
-        <geometry>
-          <mesh filename="package://ur_description/meshes/ur3/collision/wrist2.stl"/>
+          <mesh filename="visual/wrist2.dae"/>
+        </geometry>
+        <material name="LightGrey">
+          <color rgba="0.7 0.7 0.7 1.0"/>
+        </material>
+      </visual>
+      <collision>
+        <geometry>
+          <mesh filename="collision/wrist2.stl"/>
         </geometry>
       </collision>
@@ -286,13 +286,13 @@
       <visual>
         <geometry>
-          <mesh filename="package://ur_description/meshes/ur3/visual/wrist3.dae"/>
-        </geometry>
-        <material name="LightGrey">
-          <color rgba="0.7 0.7 0.7 1.0"/>
-        </material>
-      </visual>
-      <collision>
-        <geometry>
-          <mesh filename="package://ur_description/meshes/ur3/collision/wrist3.stl"/>
+          <mesh filename="visual/wrist3.dae"/>
+        </geometry>
+        <material name="LightGrey">
+          <color rgba="0.7 0.7 0.7 1.0"/>
+        </material>
+      </visual>
+      <collision>
+        <geometry>
+          <mesh filename="collision/wrist3.stl"/>
         </geometry>
       </collision>
